File: schematic/keystroke.kicad_sch (KiCad schematic)
At the start: 8 parts, among them J1 Conn_01x14_Pin, SW1 SW_Push, SW2 SW_Push, SW3 SW_Push, SW4 SW_Push, U1 PAM8403D

Commit message: finished schematic
Parts:
- added J2: Conn_01x04_Pin, symbol Connector:Conn_01x04_Pin
Connections:
- net +3V3: now also J2.3 (Pin_3)
- net GND: now also U1.11 (GND), J2.4 (Pin_4)
- net BTN_A: now reaches SW1.1
- net BTN_A: now also A1.1 (GPIO0)
- net BTN_D: now reaches SW4.1
- net BTN_D: now also A1.5 (GPIO3)
- net BTN_C: now reaches SW3.1
- net BTN_C: now also A1.4 (GPIO2)
- net VBUS: now reaches U1.6 (VDD)
- net AUDIO: now reaches U1.7 (INL)
- net AUDIO: now also A1.29 (GPIO22)
- net BTN_B: now reaches A1.2 (GPIO1)
- net BTN_B: now also SW2.1
- net CLK: now reaches A1.6 (GPIO4)
- net CLK: now also J2.1 (Pin_1)
- net DIO: now reaches A1.7 (GPIO5)
- net DIO: now also J2.2 (Pin_2)
- no-connect marks 12 -> 13
